File: Pendulum-Lamp Eagle Board/Pendulum Lamp PCB.sch (EAGLE design)
At the start: 16 parts, among them IC1 LM324N, IC2 7805TV, IC3 LM324N, IC4 7805TV, X1 2514-

Commit message: Sensor Array finished
Added sensor array in Eagle and DXF
Parts:
- added R10, R12, R14, R16, R18, R4, R6, R8: 330, rcl:R-US_0204/7
- added R11, R13, R15, R17, R19, R5, R7, R9: 10k, rcl:R-US_0204/7
- added U1, U2, U3, U4, U5, U6, U7, U8: QRD1114, SparkFun-Sensors:QRD1114
- added X2: 2514-, con-3m:2514-
Connections:
- new net GND_2: U1.E, U1.K, U2.E, U2.K, U3.E, U3.K, U4.E, U4.K, U5.E, U5.K, U6.E, U6.K, U7.E, U7.K, U8.E, U8.K, X2-2.KL
- new net N$30: R4.1, U1.A
- new net N$31: R5.1, U1.C, X2-14.KL
- new net N$34: R6.1, U2.A
- new net N$36: R7.1, U2.C, X2-13.KL
- new net N$38: R8.1, U3.A
- new net N$40: R9.1, U3.C, X2-11.KL
- new net N$42: R10.1, U4.A
- new net N$44: R11.1, U4.C, X2-9.KL
- new net N$46: R12.1, U5.A
- new net N$48: R13.1, U5.C, X2-7.KL
- new net N$50: R14.1, U6.A
- new net N$52: R15.1, U6.C, X2-5.KL
- new net N$54: R16.1, U7.A
- new net N$56: R17.1, U7.C, X2-3.KL
- new net N$58: R18.1, U8.A
- new net N$60: R19.1, U8.C, X2-1.KL
- new net VCC_2: R10.2, R11.2, R12.2, R13.2, R14.2, R15.2, R16.2, R17.2, R18.2, R19.2, R4.2, R5.2, R6.2, R7.2, R8.2, R9.2, X2-4.KL
