File: Pendulum-Lamp Eagle Board - Shield/Pendulum Lamp PCB.brd (EAGLE design)
At the start: 70.5 x 88.6 mm, 16 parts, among them IC1 LM324N, IC2 7805TV, IC3 LM324N, IC4 7805TV, X1 2514-

Commit message: First succesful model
Parts:
- moved C1 193.7 mm to (61.6, 15.2)
- moved C2 193.7 mm to (56.5, 15.2)
- moved C4 193.7 mm to (50.2, 66.0)
- moved IC1 193.7 mm to (28.6, 47.6)
- moved IC2 193.7 mm to (59.1, 4.45)
- moved IC3 193.7 mm to (28.6, 21.0)
- moved IC4 193.7 mm to (47.6, 78.1)
- moved J1 193.7 mm to (38.1, 67.9)
- moved J2 193.7 mm to (64.1, 66.7)
- moved R1 193.7 mm to (17.8, 81.3)
- moved R3 193.7 mm to (28.6, 77.5)
- moved U$1 193.7 mm to (55.2, 48.9)
- moved X1 193.7 mm to (9.53, 34.9)
- moved C3 193.7 mm to (45.1, 66.0)
- moved CN1 193.7 mm to (73.0, 79.4)
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